Commit message: Add URDF file for Franka Emika teleoperation robot configuration

File: gello/factr/urdf/GELLO_Assembly_URDF_V4/GELLO_Assembly_URDF_V4.urdf (robot description, URDF)
Before this commit: robot GELLO_Assembly_URDF_V4, 8 links, 7 joints
Joints:
- joint base_link_joint_1: limit (none) -> lower=-3.14159 upper=3.14159 effort=10 velocity=10; type continuous -> revolute
- joint link_2_joint_2: limit (none) -> lower=-3.14159 upper=3.14159 effort=10 velocity=10; type continuous -> revolute
- joint link_2_joint_3: limit (none) -> lower=-3.14159 upper=3.14159 effort=10 velocity=10; type continuous -> revolute
- joint link_3_joint_4: limit (none) -> lower=-3.14159 upper=3.14159 effort=10 velocity=10; type continuous -> revolute
- joint link_4_joint_5: limit (none) -> lower=-3.14159 upper=3.14159 effort=10 velocity=10; type continuous -> revolute
- joint link_5_joint_6: limit (none) -> lower=-3.14159 upper=3.14159 effort=10 velocity=10; type continuous -> revolute
- joint link_6_handle_gripper: limit (none) -> lower=-3.14159 upper=3.14159 effort=10 velocity=10; type continuous -> revolute

Commit message: Update configuration files and add inertia calculation script for improved robot dynamics

File: gello/factr/urdf/GELLO_Assembly_URDF_V4/GELLO_Assembly_URDF_V4.urdf (robot description, URDF)
Before this commit: robot GELLO_Assembly_URDF_V4, 8 links, 7 joints
Joints:
- joint base_link_joint_1: limit lower=-3.14159 upper=3.14159 effort=10 velocity=10 -> lower=-3.14159 upper=3.14159 effort=1.0 velocity=10
- joint link_2_joint_2: axis -1.7516230804060213e-46 -2.2402855000298757e-59 -1.0 -> 0.0 -0.0 -1.0; limit lower=-3.14159 upper=3.14159 effort=10 velocity=10 -> lower=-3.14159 upper=3.14159 effort=3.5 velocity=10
- joint link_2_joint_3: axis -1.7516230804060213e-46 -2.2402855000298757e-59 -1.0 -> 0.0 -0.0 -1.0; limit lower=-3.14159 upper=3.14159 effort=10 velocity=10 -> lower=-3.14159 upper=3.14159 effort=3.5 velocity=10
- joint link_3_joint_4: axis 0.0 1.89326617253043e-29 -1.0 -> 0.0 0.0 -1.0; limit lower=-3.14159 upper=3.14159 effort=10 velocity=10 -> lower=-3.14159 upper=3.14159 effort=1.0 velocity=10; origin xyz=0.19610000999999996 0.0 -0.025975 rpy=3.141592653589793 1.7516230804060213e-46 -1.9446922743316068e-62 -> xyz=0.19610000999999996 0.0 -0.025975 rpy=3.141592653589793 0.0 -0.0
- joint link_4_joint_5: axis -1.0 1.8611098538172282e-45 -2.2420775429197073e-44 -> -1.0 0.0 -0.0; limit lower=-3.14159 upper=3.14159 effort=10 velocity=10 -> lower=-3.14159 upper=3.14159 effort=1.0 velocity=10; origin xyz=-0.01239999999999995 0.0 -0.0425 rpy=1.89326617253043e-29 2.0090370659089317e-74 -1.0611487677000899e-45 -> xyz=-0.01239999999999995 0.0 -0.0425 rpy=0.0 0.0 -0.0
- joint link_5_joint_6: axis -0.0 -3.538195747044105e-48 -1.0 -> -0.0 -0.0 -1.0; limit lower=-3.14159 upper=3.14159 effort=10 velocity=10 -> lower=-3.14159 upper=3.14159 effort=1.0 velocity=10; origin xyz=-0.035500000000000045 0.0 -0.012000000000000002 rpy=3.538195747044105e-48 -0.0 1.0611487677000899e-45 -> xyz=-0.035500000000000045 0.0 -0.012000000000000002 rpy=0.0 -0.0 0.0
- joint link_6_handle_gripper: axis -1.0 0.0 -5.577493118932647e-31 -> -1.0 0.0 -0.0; limit lower=-3.14159 upper=3.14159 effort=10 velocity=10 -> lower=-3.14159 upper=3.14159 effort=1.0 velocity=10
