Commit message: Reworked URDFs as much as possible

File: gello/factr/urdf/GELLO_Assembly_URDF_V4/GELLO_Assembly_URDF_V4 copy.urdf (robot description, URDF)
Before this commit: robot GELLO_Assembly_URDF_V4, 8 links, 7 joints
Links:
- link base_link: mass 0.1521 -> 1.2534950685370367
- link link_1: mass 0.01753 -> 0.08462228507878798
- link link_2: mass 0.2561 -> 0.5107989598000147
- link link_3: mass 0.1353 -> 0.27478429725563525
- link link_4: mass 0.0412 -> 0.031008776139393332
- link link_5: mass 0.037 -> 0.02262454140363734
- link link_6_handle: mass 0.0482 -> 0.06041132273561478
- link link_7_trigger: mass 0.01 -> 0.009306476615493822
Joints:
- joint base_link_joint_1: limit lower=-3.14159 upper=3.14159 effort=1.0 velocity=10 -> (none); type revolute -> continuous
- joint link_2_joint_2: axis 0.0 -0.0 -1.0 -> -1.7516230804060213e-46 -2.2402855000298757e-59 -1.0; child link_2 -> link_1; limit lower=-3.14159 upper=3.14159 effort=3.5 velocity=10 -> (none); parent link_1 -> link_2; type revolute -> continuous
- joint link_2_joint_3: axis 0.0 -0.0 -1.0 -> -1.7516230804060213e-46 -2.2402855000298757e-59 -1.0; limit lower=-3.14159 upper=3.14159 effort=3.5 velocity=10 -> (none); type revolute -> continuous
- joint link_3_joint_4: axis 0.0 0.0 -1.0 -> 0.0 1.89326617253043e-29 -1.0; limit lower=-3.14159 upper=3.14159 effort=1.0 velocity=10 -> (none); origin xyz=0.19610000999999996 0.0 -0.025975 rpy=3.141592653589793 0.0 -0.0 -> xyz=0.19610000999999996 0.0 -0.025975 rpy=3.141592653589793 1.7516230804060213e-46 -1.9446922743316068e-62; type revolute -> continuous
- joint link_4_joint_5: axis -1.0 0.0 -0.0 -> -1.0 1.8611098538172282e-45 -2.2420775429197073e-44; limit lower=-3.14159 upper=3.14159 effort=1.0 velocity=10 -> (none); origin xyz=-0.01239999999999995 0.0 -0.0425 rpy=0.0 0.0 -0.0 -> xyz=-0.01239999999999995 0.0 -0.0425 rpy=1.89326617253043e-29 2.0090370659089317e-74 -1.0611487677000899e-45; type revolute -> continuous
- joint link_5_joint_6: axis -0.0 -0.0 -1.0 -> -0.0 -3.538195747044105e-48 -1.0; limit lower=-3.14159 upper=3.14159 effort=1.0 velocity=10 -> (none); origin xyz=-0.035500000000000045 0.0 -0.012000000000000002 rpy=0.0 -0.0 0.0 -> xyz=-0.035500000000000045 0.0 -0.012000000000000002 rpy=3.538195747044105e-48 -0.0 1.0611487677000899e-45; type revolute -> continuous
- joint link_6_handle_gripper: axis -1.0 0.0 -0.0 -> -1.0 0.0 -5.577493118932647e-31; limit lower=-3.14159 upper=3.14159 effort=1.0 velocity=10 -> (none); type revolute -> continuous
