Commit message: Add gravity torque testing, setup validation, and URDF visualization scripts
- Implemented `test_gravity_torques.py` for real-time gravity torque testing with Dynamixel motors.
- Created `validate_gello_setup.py` to validate the GELLO setup, including URDF loading, Dynamixel connectivity, calibration, and torque mapping.
- Developed `visualize_leader_urdf_meshcat.py` to visualize real leader joint angles against the URDF using MeshCat.
- Enhanced calibration methods and added detailed logging for diagnostics.
- Included error handling and configuration checks for improved robustness.

File: gello/factr/urdf/GELLO_Assembly_URDF_V4/GELLO_Assembly_URDF_V4_changedFrame.urdf (robot description, URDF)
Before this commit: robot GELLO_Assembly_URDF_V4, 9 links, 8 joints
Links:
- link base_link: geometry collision mesh filename=meshes/base_link.stl scale=0.001 0.001 0.001; visual box size=0.003 0.003 0.05
- link link_1: geometry collision mesh filename=meshes/link_1.stl scale=0.001 0.001 0.001; visual box size=0.003 0.003 0.05
- link link_2: geometry collision mesh filename=meshes/link_2.stl scale=0.001 0.001 0.001; visual box size=0.003 0.003 0.05
- link link_3: geometry collision mesh filename=meshes/link_3.stl scale=0.001 0.001 0.001; visual box size=0.003 0.003 0.05
- link link_4: geometry collision mesh filename=meshes/link_4.stl scale=0.001 0.001 0.001; visual box size=0.003 0.003 0.05
- link link_5: geometry collision mesh filename=meshes/link_5.stl scale=0.001 0.001 0.001; visual box size=0.003 0.003 0.05
- link link_6_handle: geometry collision mesh filename=meshes/link_6_handle.stl scale=0.001 0.001 0.001; visual box size=0.003 0.003 0.05
- link link_7_trigger: geometry collision mesh filename=meshes/link_7_trigger.stl scale=0.001 0.001 0.001; visual box size=0.003 0.003 0.05

File: gello/factr/urdf/GELLO_Assembly_URDF_V4/GELLO_Assembly_URDF_V4_changedFrame_J3minusZ.urdf (robot description, URDF)
Before this commit: robot GELLO_Assembly_URDF_V4, 9 links, 8 joints
Links:
- link base_link: geometry collision mesh filename=meshes/base_link.stl scale=0.001 0.001 0.001; visual box size=0.003 0.003 0.05
- link link_1: geometry collision mesh filename=meshes/link_1.stl scale=0.001 0.001 0.001; visual box size=0.003 0.003 0.05
- link link_2: geometry collision mesh filename=meshes/link_2.stl scale=0.001 0.001 0.001; visual box size=0.003 0.003 0.05
- link link_3: geometry collision mesh filename=meshes/link_3.stl scale=0.001 0.001 0.001; visual box size=0.003 0.003 0.05
- link link_4: geometry collision mesh filename=meshes/link_4.stl scale=0.001 0.001 0.001; visual box size=0.003 0.003 0.05
- link link_5: geometry collision mesh filename=meshes/link_5.stl scale=0.001 0.001 0.001; visual box size=0.003 0.003 0.05
- link link_6_handle: geometry collision mesh filename=meshes/link_6_handle.stl scale=0.001 0.001 0.001; visual box size=0.003 0.003 0.05
- link link_7_trigger: geometry collision mesh filename=meshes/link_7_trigger.stl scale=0.001 0.001 0.001; visual box size=0.003 0.003 0.05
Joints:
- joint link_2_joint_3: axis 1.0 0.0 0.0 -> 0.0 -0.0 -1.0

File: gello/factr/urdf/GELLO_Assembly_URDF_V4/GELLO_Assembly_URDF_V4_noGripper.urdf (robot description, URDF)
Before this commit: robot GELLO_Assembly_URDF_V4, 9 links, 8 joints
Links:
- removed link link_2_extra_mass
- removed link link_7_trigger
- link link_2: mass 0.45 -> 0.2561
- link link_3: mass 0.25 -> 0.1353
Joints:
- removed joint link_2_extra_mass_joint
- removed joint link_6_handle_gripper
- joint link_2_joint_3: axis 1.0 0.0 0.0 -> 0.0 -0.0 -1.0
